File: PCB/acoustic_levitation_main.kicad_pcb (KiCad board)
At the start: 2 copper layers, 88 x 88 mm, 68 parts, among them J1 DE0-Nano-SoC: GPIO 0, J10 PJ-102AH, J2 DE0-Nano-SoC: GPIO 1, J3 DE0-Nano-SoC: JP3, J4 DE0-Nano-SoC: JP2, J5 DE0-Nano-SoC: JP5[3], J6 8-215079-8, J7 8-215079-8, J8 8-215079-8, J9 8-215079-8, Q1 Si3421DV, U1 MAX17079, U2 MAX17079, U3 MAX17079, U4 MAX17079, U5 MAX17079, U6 MAX17079, U7 TSR2-2450

Commit message: Upgraded PCB to KiCad 5
Parts:
- C1, C10, C11, C12, C2, C3, C4, C5, C6, C7, C8, C9: footprint Capacitors_SMD:C_0805_HandSoldering -> footprints:C_0805_HandSoldering
- J1, J2: footprint Socket_Strips:Socket_Strip_Straight_2x20_Pitch2.54mm -> footprints:Socket_Strip_Straight_2x20_Pitch2.54mm
- J3: footprint Pin_Headers:Pin_Header_Straight_1x08_Pitch2.54mm -> footprints:Pin_Header_Straight_1x08_Pitch2.54mm
- J4: footprint Pin_Headers:Pin_Header_Straight_1x10_Pitch2.54mm -> footprints:Pin_Header_Straight_1x10_Pitch2.54mm
- J5: footprint Pin_Headers:Pin_Header_Straight_1x01_Pitch2.54mm -> footprints:Pin_Header_Straight_1x01_Pitch2.54mm
