File: PCB/acoustic_levitation_wing.kicad_pcb (KiCad board)
At the start: 2 copper layers, 98.8 x 24 mm, 22 parts, among them J1 8-215079-8, U1 MAX17079, U2 MAX17079

Commit message: Upgraded PCB to KiCad 5
Parts:
- C1, C2, C3, C4: footprint Capacitors_SMD:C_0805_HandSoldering -> footprints:C_0805_HandSoldering
