File: PCB/acoustic_levitation_wing.sch (KiCad schematic (older format))
At the start: 1 part, among them J1 8-215079-8

Commit message: Upgraded PCB to KiCad 5
Parts:
- J1: symbol Conn_02x09_Odd_Even -> Connector_Generic:Conn_02x09_Odd_Even
Changed lines of the file:
@@
-EESchema Schematic File Version 2
-LIBS:power
-LIBS:device
-LIBS:transistors
-LIBS:conn
-LIBS:linear
-LIBS:regul
-LIBS:74xx
-LIBS:cmos4000
-LIBS:adc-dac
-LIBS:memory
-LIBS:xilinx
-LIBS:microcontrollers
-LIBS:dsp
-LIBS:microchip
-LIBS:analog_switches
-LIBS:motorola
-LIBS:texas
-LIBS:intel
-LIBS:audio
-LIBS:interface
-LIBS:digital-audio
-LIBS:philips
-LIBS:display
-LIBS:cypress
-LIBS:siliconi
-LIBS:opto
-LIBS:atmel
-LIBS:contrib
-LIBS:valves
-LIBS:library
+EESchema Schematic File Version 4
 LIBS:acoustic_levitation_wing-cache
-EELAYER 25 0
+EELAYER 26 0
 EELAYER END
 $Descr A4 11693 8268
@@
 $EndSheet
 $Comp
-L Conn_02x09_Odd_Even J1
+L Connector_Generic:Conn_02x09_Odd_Even J1
 U 1 1 5AB0F29A
 P 5600 3150
@@
 	5300 3550 5300 3650
 $Comp
-L GND #PWR01
+L power:GND #PWR01
 U 1 1 5AB0F821
 P 5300 3650
@@
 Enable
 $Comp
-L +12V #PWR02
+L power:+12V #PWR02
 U 1 1 5AB0F8BD
 P 6300 3450
@@
 $EndComp
 $Comp
-L +3V3 #PWR03
+L power:+3V3 #PWR03
 U 1 1 5AB0F918
 P 6300 3550
