File: PCB/piezo_x7.sch (KiCad schematic (older format))
At the start: 10 parts, among them U1 MAX17079

Commit message: Upgraded PCB to KiCad 5
Parts:
- C1, C2: footprint Capacitors_SMD:C_0805_HandSoldering -> footprints:C_0805_HandSoldering; symbol C -> Device:C
- TR1, TR2, TR3, TR4, TR5, TR6, TR7: symbol MA40S4S -> library:MA40S4S
- U1: symbol MAX17079 -> library:MAX17079
