File: PCB/power.sch (KiCad schematic (older format))
At the start: 3 parts, among them J10 PJ-102AH, Q1 Si3421DV, U7 TSR2-2450

Commit message: Upgraded PCB to KiCad 5
Parts:
- J10: symbol Barrel_Jack -> Connector:Barrel_Jack_Switch
- Q1: symbol Si3421DV -> library:Si3421DV
- U7: symbol TSR2-2450 -> library:TSR2-2450
Changed lines of the file:
@@
-EESchema Schematic File Version 2
-LIBS:power
-LIBS:device
-LIBS:switches
-LIBS:relays
-LIBS:motors
-LIBS:transistors
-LIBS:conn
-LIBS:linear
-LIBS:regul
-LIBS:74xx
-LIBS:cmos4000
-LIBS:adc-dac
-LIBS:memory
-LIBS:xilinx
-LIBS:microcontrollers
-LIBS:dsp
-LIBS:microchip
-LIBS:analog_switches
-LIBS:motorola
-LIBS:texas
-LIBS:intel
-LIBS:audio
-LIBS:interface
-LIBS:digital-audio
-LIBS:philips
-LIBS:display
-LIBS:cypress
-LIBS:siliconi
-LIBS:opto
-LIBS:atmel
-LIBS:contrib
-LIBS:valves
-LIBS:library
+EESchema Schematic File Version 4
 LIBS:acoustic_levitation_main-cache
-EELAYER 25 0
+EELAYER 26 0
 EELAYER END
 $Descr A4 11693 8268
@@
 $EndDescr
 $Comp
-L GND #PWR064
+L power:GND #PWR064
 U 1 1 5AAB1DD3
 P 5100 3700
@@
 $EndComp
 $Comp
-L +12V #PWR065
+L power:+12V #PWR065
 U 1 1 5AAB1DEA
 P 5700 3050
@@
 $EndComp
 $Comp
-L GND #PWR066
+L power:GND #PWR066
 U 1 1 5AAA7C9E
 P 6300 3700
@@
 $EndComp
 $Comp
-L Barrel_Jack J10
+L Connector:Barrel_Jack_Switch J10
 U 1 1 5AAAC0A9
 P 4700 3350
 F 0 "J10" H 4700 3560 50  0000 C CNN
-F 1 "PJ-102AH" H 4700 3175 50  0000 C CNN
+F 1 "PJ-102AH" H 4700 3150 50  0000 C CNN
 F 2 "footprints:CUI_PJ-102AH" H 4750 3310 50  0001 C CNN
 F 3 "" H 4750 3310 50  0001 C CNN
@@
 $EndComp
 $Comp
-L +5V #PWR067
+L power:+5V #PWR067
 U 1 1 5AABB86C
 P 6900 3050
@@
 $EndComp
 $Comp
-L GND #PWR068
+L power:GND #PWR068
 U 1 1 5AB62943
 P 5400 3700
@@
 $EndComp
 Wire Wire Line
-	5600 3250 5800 3250
+	5600 3250 5700 3250
 Wire Wire Line
 	5700 3250 5700 3050
@@
 	5000 3350 5100 3350
 Wire Wire Line
-	5100 3350 5100 3700
+	5100 3350 5100 3450
 Connection ~ 5700 3250
 Wire Wire Line
@@
 Connection ~ 5100 3450
 Wire Wire Line
-	5000 3250 5200 3250
+	5000 3250 5100 3250
 Wire Wire Line
 	5400 3550 5400 3700
 $Comp
-L +VDC #PWR069
+L power:+VDC #PWR069
 U 1 1 5AB6380E
 P 5100 3150
@@
 Connection ~ 5100 3250
 $Comp
-L Si3421DV Q1
+L library:Si3421DV Q1
 U 1 1 5AC4DD7C
 P 5400 3350
@@
 F 2 "footprints:TSOP-6_2.9x1.5mm_Pitch0.95mm" H 5600 3200 50  0001 L CNN
 F 3 "http://www.vishay.com/docs/62921/si3421dv.pdf" H 5600 3100 50  0001 L CNN
-F 4 "Digi-Key" H 5600 2900 50  0001 L CNN "Supplier1"
+F 4 "Vishay Siliconix" H 5600 3000 50  0001 L CNN "Manufacturer"
 F 5 "SI3421DV-T1-GE3" H 6250 3000 50  0001 L CNN "ManufacturerPartNumber"
-F 6 "SI3421DV-T1-GE3CT-ND" H 6000 2900 50  0001 L CNN "Supplier1PartNumber"
-F 7 "Vishay Siliconix" H 5600 3000 50  0001 L CNN "Manufacturer"
+F 6 "Digi-Key" H 5600 2900 50  0001 L CNN "Supplier1"
+F 7 "SI3421DV-T1-GE3CT-ND" H 6000 2900 50  0001 L CNN "Supplier1PartNumber"
 	1    5400 3350
 	0    -1   -1   0
 $EndComp
 $Comp
-L TSR2-2450 U7
+L library:TSR2-2450 U7
 U 1 1 5AC4DDD8
 P 6300 3350
@@
 F 2 "footprints:Traco_TSR2" H 6350 3000 50  0001 L CNN
 F 3 "https://assets.tracopower.com/TSR2/documents/tsr2-datasheet.pdf" H 6350 2900 50  0001 L CNN
-F 4 "300-67-301" H 6750 2600 50  0001 L CNN "Supplier2PartNumber"
-F 5 "495-TSR2-2450" H 6650 2700 50  0001 L CNN "Supplier1PartNumber"
-F 6 "Distrelec" H 6350 2600 50  0001 L CNN "Supplier2"
-F 7 "Mouser" H 6350 2700 50  0001 L CNN "Supplier1"
-F 8 "Traco Power" H 6350 2800 50  0001 L CNN "Manufacturer"
-F 9 "TSR 2-2450" H 6850 2800 50  0001 L CNN "ManufacturerPartNumber"
+F 4 "Traco Power" H 6350 2800 50  0001 L CNN "Manufacturer"
+F 5 "TSR 2-2450" H 6850 2800 50  0001 L CNN "ManufacturerPartNumber"
+F 6 "Mouser" H 6350 2700 50  0001 L CNN "Supplier1"
+F 7 "495-TSR2-2450" H 6650 2700 50  0001 L CNN "Supplier1PartNumber"
+F 8 "Distrelec" H 6350 2600 50  0001 L CNN "Supplier2"
+F 9 "300-67-301" H 6750 2600 50  0001 L CNN "Supplier2PartNumber"
 	1    6300 3350
 	1    0    0    -1
 $EndComp
+Wire Wire Line
+	5700 3250 5800 3250
+Wire Wire Line
+	5100 3450 5100 3700
+Wire Wire Line
+	5100 3250 5200 3250
 $EndSCHEMATC
